File: PCB/Chirstmas-Card.kicad_pcb (KiCad board)
At the start: 2 copper layers, 105 x 148 mm, 100 parts, among them J1 Conn_ARM_SWD_TagConnect_TC203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, SW1 SW_SPST, SW2 SW_SPST, SW3 SW_SPST, U1 PAM8904EGPR, U2 STM32G030C6Tx, Y1 Crystal

Commit message: Added initial buzzer functionality
Parts:
- removed C1, C2: 10uF, Capacitor_SMD:C_0603_1608Metric
- removed C3, C4: 1uF, Capacitor_SMD:C_0603_1608Metric
- removed R1, R2, R3, R4, R5, R6, R7, R8: 0, Resistor_SMD:R_0402_1005Metric
- removed R10, R11, R15, R16: 0r, Resistor_SMD:R_0402_1005Metric
- removed R14: 100k, Resistor_SMD:R_0402_1005Metric
- removed U1: PAM8904EGPR, EN_Designs-Footprints:QFN50P300X300X100-13N
- added ?: , , F.Cu at (43.0, 175.0)
- added ?: , , F.Cu at (43.0, 33.0)
- added Art: Val**, EN_Designs-Footprints:jordi-christmas-girl, F.Cu at (-99.1, 104.3)
- added Art: Val**, EN_Designs-Footprints:jordi-christmas-girl, F.Cu at (92.5, 104.0)
- added REF**: JLC_PCB_Tooling_Hole, EN_Designs-Footprints:JLC_PCB_Tooling_Hole, F.Cu at (143.0, 33.0)
- BT1, C10, C11, C5, C6, C7, C8, C9, J1, LS1, U2, Y1: moved to B.Cu
- D1, D10, D11, D12, D13, D14, D15, D16, D17, D18, D19, D2, D20, D21, D22, D23, D24, D25, D26, D27, D28, D29, D3, D30, D31, D32, D33, D34, D35, D36, D37, D38, D39, D4, D40, D41, D42, D43, D44, D45, D46, D47, D48, D49, D5, D50, D51, D52, D53, D54, D55, D56, D57, D58, D59, D6, D60, D61, D62, D63, D64, D7, D8, D9: footprint LED_SMD:LED_0805_2012Metric -> EN_Designs-Footprints:MHT151WDT; moved to B.Cu
- R12, R13, R9: footprint Resistor_SMD:R_0402_1005Metric -> Resistor_SMD:R_0603_1608Metric; moved to B.Cu
- moved J1 93.3 mm to (138.8, 173.7), turned to 180 degrees
- moved R13 67.3 mm to (78.1, 58.6)
- moved C5 67.2 mm to (77.3, 44.4), turned to 180 degrees
- moved C6 67.2 mm to (77.3, 46.9), turned to 180 degrees
- moved R12 64.8 mm to (77.5, 61.1)
- moved Y1 62.8 mm to (79.8, 45.6)
- moved R9 62.7 mm to (76.6, 63.5)
- moved C9 53.9 mm to (83.8, 44.8)
- moved C8 52.0 mm to (84.8, 44.8)
- moved U2 51.3 mm to (85.2, 51.2)
- moved C10 49.4 mm to (86.3, 45.3), turned to 0 degrees
- moved C11 48.3 mm to (86.9, 44.0), turned to 0 degrees
- moved C7 44.4 mm to (89.0, 45.2), turned to 0 degrees
- moved LS1 43.8 mm to (68.5, 50.5), turned to 0 degrees
- moved D15 43.4 mm to (129.0, 66.0), turned to -135 degrees
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Connections:
- D1 pad 2: Net-(D1-A) -> /C6
- D10 pad 2: Net-(D10-A) -> /C5
- D11 pad 2: Net-(D11-A) -> /C4
- D12 pad 2: Net-(D12-A) -> /C3
- D13 pad 2: Net-(D13-A) -> /C2
- D14 pad 2: Net-(D14-A) -> /C1
- D15 pad 2: Net-(D15-A) -> /C8
- D16 pad 2: Net-(D16-A) -> /C7
- D17 pad 2: Net-(D1-A) -> /C6
- D18 pad 2: Net-(D10-A) -> /C5
- D19 pad 2: Net-(D11-A) -> /C4
- D2 pad 2: Net-(D10-A) -> /C5
- D20 pad 2: Net-(D12-A) -> /C3
- D21 pad 2: Net-(D13-A) -> /C2
- D22 pad 2: Net-(D14-A) -> /C1
- D23 pad 2: Net-(D15-A) -> /C8
- D24 pad 2: Net-(D16-A) -> /C7
- D25 pad 2: Net-(D1-A) -> /C6
- D26 pad 2: Net-(D10-A) -> /C5
- D27 pad 2: Net-(D11-A) -> /C4
- D28 pad 2: Net-(D12-A) -> /C3
- D29 pad 2: Net-(D13-A) -> /C2
- D3 pad 2: Net-(D11-A) -> /C4
- D30 pad 2: Net-(D14-A) -> /C1
- D31 pad 2: Net-(D15-A) -> /C8
- D32 pad 2: Net-(D16-A) -> /C7
- D33 pad 2: Net-(D1-A) -> /C6
- D34 pad 2: Net-(D10-A) -> /C5
- D35 pad 2: Net-(D11-A) -> /C4
- D36 pad 2: Net-(D12-A) -> /C3
- D37 pad 2: Net-(D13-A) -> /C2
- D38 pad 2: Net-(D14-A) -> /C1
- D39 pad 2: Net-(D15-A) -> /C8
- D4 pad 2: Net-(D12-A) -> /C3
- D40 pad 2: Net-(D16-A) -> /C7
- D41 pad 2: Net-(D1-A) -> /C6
- D42 pad 2: Net-(D10-A) -> /C5
- D43 pad 2: Net-(D11-A) -> /C4
- D44 pad 2: Net-(D12-A) -> /C3
- D45 pad 2: Net-(D13-A) -> /C2
- D46 pad 2: Net-(D14-A) -> /C1
- D47 pad 2: Net-(D15-A) -> /C8
- D48 pad 2: Net-(D16-A) -> /C7
- D49 pad 2: Net-(D1-A) -> /C6
- D5 pad 2: Net-(D13-A) -> /C2
- D50 pad 2: Net-(D10-A) -> /C5
- D51 pad 2: Net-(D11-A) -> /C4
- D52 pad 2: Net-(D12-A) -> /C3
- D53 pad 2: Net-(D13-A) -> /C2
- D54 pad 2: Net-(D14-A) -> /C1
- D55 pad 2: Net-(D15-A) -> /C8
- D56 pad 2: Net-(D16-A) -> /C7
- D57 pad 2: Net-(D1-A) -> /C6
- D58 pad 2: Net-(D10-A) -> /C5
- D59 pad 2: Net-(D11-A) -> /C4
- D6 pad 2: Net-(D14-A) -> /C1
- D60 pad 2: Net-(D12-A) -> /C3
- D61 pad 2: Net-(D13-A) -> /C2
- D62 pad 2: Net-(D14-A) -> /C1
- D63 pad 2: Net-(D15-A) -> /C8
- D64 pad 2: Net-(D16-A) -> /C7
- D7 pad 2: Net-(D15-A) -> /C8
- D8 pad 2: Net-(D16-A) -> /C7
- D9 pad 2: Net-(D1-A) -> /C6
- LS1 pad 1: Net-(U1-VO1) -> Net-(U2-PB3)
- LS1 pad 2: Net-(U1-VO2) -> Net-(U2-PB6)
- U2 pad 15: /BUZZER -> unconnected-(U2-PA4-Pad15)
- U2 pad 17: /C1 -> /C8
- U2 pad 18: /C2 -> /C7
- U2 pad 19: /C3 -> /C6
- U2 pad 20: /C4 -> /C5
- U2 pad 21: /C5 -> /C4
- U2 pad 22: /C6 -> /C3
- U2 pad 23: /C7 -> /C2
- U2 pad 24: /C8 -> /C1
- U2 pad 37: /BTN1 -> /BTN3
- U2 pad 39: /BTN3 -> /BTN1
- U2 pad 42: unconnected-(U2-PB3-Pad42) -> Net-(U2-PB3)
- U2 pad 45: unconnected-(U2-PB6-Pad45) -> Net-(U2-PB6)
Routing:
- net VCC: track 83.6 -> 284.3 mm, vias 5 -> 0
- net /RESET: track 22.1 -> 161.8 mm, vias 2 -> 0
- net /SWCLK: track 7.27 -> 141.0 mm
- net /SWDIO: track 8.74 -> 141.3 mm
- net /C8: track 5.58 -> 93.5 mm, vias 0 -> 9
- net /C7: track 11.1 -> 88.3 mm, vias 0 -> 9
- net /C6: track 16.6 -> 83.1 mm, vias 0 -> 9
- net /C5: track 22.1 -> 77.9 mm, vias 0 -> 9
- net Net-(D15-A): track 54.4 -> 0.00 mm, vias 9 -> 0
- net Net-(D16-A): track 54.4 -> 0.00 mm, vias 9 -> 0
- net Net-(D14-A): track 54.4 -> 0.00 mm, vias 9 -> 0
- net Net-(D12-A): track 54.4 -> 0.00 mm, vias 9 -> 0
- net Net-(D11-A): track 54.4 -> 0.00 mm, vias 9 -> 0
- net Net-(D10-A): track 54.4 -> 0.00 mm, vias 9 -> 0
- net Net-(D13-A): track 54.3 -> 0.00 mm, vias 9 -> 0
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- removed copper zone on F.Cu, net GND
Other:
- board size 105 x 148 mm -> 106 x 148 mm
- board text added: "Battery model: CR2032 Insert with larger side up!"
- board text added: "Electronic card 2024 V1 Art: Jordi Navarrete Electronics: Eric Navarrete"

Commit message: -migration to new cube mx version and cmake toolchain
Parts:
- removed the Art at (-99.1, 104.3)
- removed the Art at (92.5, 104.0)
- removed R13, R9: 100k, Resistor_SMD:R_0603_1608Metric
- added Art: Val**, EN_Designs-Footprints:jordi-christmas-girl-V2, F.Cu at (93.0, 104.0)
- added R4: 0, Resistor_SMD:R_0603_1608Metric, B.Cu at (73.7, 47.0)
- added R5: 0, Resistor_SMD:R_0603_1608Metric, B.Cu at (83.7, 39.8)
- moved ? 173.7 mm to (143.0, 175.0)
- moved J1 167.3 mm to (45.0, 35.1), turned to -45 degrees
- moved D16 35.7 mm to (129.7, 65.8)
- moved D24 35.7 mm to (129.7, 70.8)
- moved D32 35.7 mm to (129.7, 75.8)
- moved D40 35.7 mm to (129.7, 80.8)
- moved D48 35.7 mm to (129.7, 85.8)
- moved D56 35.7 mm to (129.7, 90.8)
- moved D64 35.7 mm to (129.7, 95.8)
- moved D8 35.7 mm to (129.7, 60.8)
- moved D17 34.3 mm to (94.7, 70.8)
- moved D25 34.3 mm to (94.7, 75.8)
- moved D33 34.3 mm to (94.7, 80.8)
- moved D41 34.3 mm to (94.7, 85.8)
- moved D49 34.3 mm to (94.7, 90.8)
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- renumbered C9 to C1, C10 to C2, C11 to C3, C8 to C4, C7 to C5, C5 to C7, D7 to D1, D16 to D10, D9 to D11, D10 to D12, D11 to D13, D12 to D14, D13 to D15, D14 to D16, D23 to D17, D24 to D18, D17 to D19, D8 to D2, D18 to D20, D19 to D21, D20 to D22, D21 to D23, D22 to D24, D31 to D25, D32 to D26, D25 to D27, D26 to D28, D27 to D29, D1 to D3, D28 to D30, D29 to D31, D30 to D32, D39 to D33, D40 to D34, D33 to D35, D34 to D36, D35 to D37, D36 to D38, D37 to D39, D2 to D4, D38 to D40, D47 to D41, D48 to D42, D41 to D43, D42 to D44, D43 to D45, D44 to D46, D45 to D47, D46 to D48, D55 to D49, D3 to D5, D56 to D50, D49 to D51, D50 to D52, D51 to D53, D52 to D54, D53 to D55, D54 to D56, D63 to D57, D64 to D58, D57 to D59, D4 to D6, D58 to D60, D59 to D61, D60 to D62, D61 to D63, D62 to D64, D5 to D7, D6 to D8, D15 to D9, R12 to R2, U2 to U1
Connections:
- D1 pad 1: /R1 -> /R0
- D1 pad 2: /C8 -> /C0
- D10 pad 1: /R2 -> /R1
- D10 pad 2: /C7 -> /C1
- D11 pad 1: /R2 -> /R1
- D11 pad 2: /C6 -> /C2
- D12 pad 1: /R2 -> /R1
- D12 pad 2: /C5 -> /C3
- D13 pad 1: /R2 -> /R1
- D14 pad 1: /R2 -> /R1
- D14 pad 2: /C3 -> /C5
- D15 pad 1: /R2 -> /R1
- D15 pad 2: /C2 -> /C6
- D16 pad 1: /R2 -> /R1
- D16 pad 2: /C1 -> /C7
- D17 pad 1: /R3 -> /R2
- D17 pad 2: /C8 -> /C0
- D18 pad 1: /R3 -> /R2
- D18 pad 2: /C7 -> /C1
- D19 pad 1: /R3 -> /R2
- D19 pad 2: /C6 -> /C2
- D2 pad 1: /R1 -> /R0
- D2 pad 2: /C7 -> /C1
- D20 pad 1: /R3 -> /R2
- D20 pad 2: /C5 -> /C3
- D21 pad 1: /R3 -> /R2
- D22 pad 1: /R3 -> /R2
- D22 pad 2: /C3 -> /C5
- D23 pad 1: /R3 -> /R2
- D23 pad 2: /C2 -> /C6
- D24 pad 1: /R3 -> /R2
- D24 pad 2: /C1 -> /C7
- D25 pad 1: /R4 -> /R3
- D25 pad 2: /C8 -> /C0
- D26 pad 1: /R4 -> /R3
- D26 pad 2: /C7 -> /C1
- D27 pad 1: /R4 -> /R3
- D27 pad 2: /C6 -> /C2
- D28 pad 1: /R4 -> /R3
- D28 pad 2: /C5 -> /C3
- D29 pad 1: /R4 -> /R3
- D3 pad 1: /R1 -> /R0
- D3 pad 2: /C6 -> /C2
- D30 pad 1: /R4 -> /R3
- D30 pad 2: /C3 -> /C5
- D31 pad 1: /R4 -> /R3
- D31 pad 2: /C2 -> /C6
- D32 pad 1: /R4 -> /R3
- D32 pad 2: /C1 -> /C7
- D33 pad 1: /R5 -> /R4
- D33 pad 2: /C8 -> /C0
- D34 pad 1: /R5 -> /R4
- D34 pad 2: /C7 -> /C1
- D35 pad 1: /R5 -> /R4
- D35 pad 2: /C6 -> /C2
- D36 pad 1: /R5 -> /R4
- D36 pad 2: /C5 -> /C3
- D37 pad 1: /R5 -> /R4
- D38 pad 1: /R5 -> /R4
- D38 pad 2: /C3 -> /C5
- D39 pad 1: /R5 -> /R4
- D39 pad 2: /C2 -> /C6
- D4 pad 1: /R1 -> /R0
- D4 pad 2: /C5 -> /C3
- D40 pad 1: /R5 -> /R4
- D40 pad 2: /C1 -> /C7
- D41 pad 1: /R6 -> /R5
- D41 pad 2: /C8 -> /C0
- D42 pad 1: /R6 -> /R5
- D42 pad 2: /C7 -> /C1
- D43 pad 1: /R6 -> /R5
- D43 pad 2: /C6 -> /C2
- D44 pad 1: /R6 -> /R5
- D44 pad 2: /C5 -> /C3
- D45 pad 1: /R6 -> /R5
- D46 pad 1: /R6 -> /R5
- D46 pad 2: /C3 -> /C5
- D47 pad 1: /R6 -> /R5
- D47 pad 2: /C2 -> /C6
- D48 pad 1: /R6 -> /R5
- D48 pad 2: /C1 -> /C7
- D49 pad 1: /R7 -> /R6
- D49 pad 2: /C8 -> /C0
- D5 pad 1: /R1 -> /R0
- D50 pad 1: /R7 -> /R6
- D50 pad 2: /C7 -> /C1
- D51 pad 1: /R7 -> /R6
- D51 pad 2: /C6 -> /C2
- D52 pad 1: /R7 -> /R6
- D52 pad 2: /C5 -> /C3
- D53 pad 1: /R7 -> /R6
- D54 pad 1: /R7 -> /R6
- D54 pad 2: /C3 -> /C5
- D55 pad 1: /R7 -> /R6
- D55 pad 2: /C2 -> /C6
- D56 pad 1: /R7 -> /R6
- D56 pad 2: /C1 -> /C7
- D57 pad 1: /R8 -> /R7
- D57 pad 2: /C8 -> /C0
- D58 pad 1: /R8 -> /R7
- D58 pad 2: /C7 -> /C1
- D59 pad 1: /R8 -> /R7
- D59 pad 2: /C6 -> /C2
- D6 pad 1: /R1 -> /R0
- D6 pad 2: /C3 -> /C5
- D60 pad 1: /R8 -> /R7
- D60 pad 2: /C5 -> /C3
- D61 pad 1: /R8 -> /R7
- D62 pad 1: /R8 -> /R7
- D62 pad 2: /C3 -> /C5
- D63 pad 1: /R8 -> /R7
- D63 pad 2: /C2 -> /C6
- D64 pad 1: /R8 -> /R7
- D64 pad 2: /C1 -> /C7
- D7 pad 1: /R1 -> /R0
- D7 pad 2: /C2 -> /C6
- D8 pad 1: /R1 -> /R0
- D8 pad 2: /C1 -> /C7
- D9 pad 1: /R2 -> /R1
- D9 pad 2: /C8 -> /C0
- J1 pad 2: /SWDIO -> Net-(J1-SWDIO)
- J1 pad 3: /RESET -> Net-(J1-~{RESET})
- LS1 pad 1: Net-(U2-PB3) -> Net-(U1-PA8)
- LS1 pad 2: Net-(U2-PB6) -> Net-(U1-PA9/NC)
- U1 pad 1: unconnected-(U2-PC13-Pad1) -> /BTN2
- U1 pad 11: unconnected-(U2-PA0-Pad11) -> /C0
- U1 pad 12: unconnected-(U2-PA1-Pad12) -> /C1
- U1 pad 13: unconnected-(U2-PA2-Pad13) -> /C2
- U1 pad 14: unconnected-(U2-PA3-Pad14) -> /C3
- U1 pad 15: unconnected-(U2-PA4-Pad15) -> /C4
- U1 pad 16: unconnected-(U2-PA5-Pad16) -> /C5
- U1 pad 17: /C8 -> /C6
- U1 pad 19: /C6 -> /R0
- U1 pad 20: /C5 -> /R1
- U1 pad 21: /C4 -> /R2
- U1 pad 22: /C3 -> unconnected-(U1-PB10-Pad22)
- U1 pad 23: /C2 -> unconnected-(U1-PB11-Pad23)
- U1 pad 24: /C1 -> unconnected-(U1-PB12-Pad24)
- U1 pad 25: /R1 -> unconnected-(U1-PB13-Pad25)
- U1 pad 26: /R2 -> unconnected-(U1-PB14-Pad26)
- U1 pad 27: /R3 -> unconnected-(U1-PB15-Pad27)
- U1 pad 28: /R4 -> Net-(U1-PA8)
- U1 pad 29: /R5 -> Net-(U1-PA9/NC)
- U1 pad 30: /R6 -> unconnected-(U1-PC6-Pad30)
- U1 pad 31: /R7 -> unconnected-(U1-PC7-Pad31)
- U1 pad 32: /R8 -> unconnected-(U1-PA10/NC-Pad32)
- U1 pad 42: Net-(U2-PB3) -> /R3
- U1 pad 43: unconnected-(U2-PB4-Pad43) -> /R4
- U1 pad 44: /BTN2 -> /R5
- U1 pad 45: Net-(U2-PB6) -> /R6
- U1 pad 46: unconnected-(U2-PB7-Pad46) -> /R7
Routing:
- net VCC: track 284.3 -> 139.4 mm
- net /SWDIO: track 141.3 -> 16.7 mm
- net /RESET: track 161.8 -> 49.0 mm
- net /C8: track 93.5 -> 0.00 mm, vias 9 -> 0
- net /SWCLK: track 141.0 -> 52.5 mm
- net /R8: track 85.1 -> 0.00 mm
- net /C0: track 0.00 -> 75.1 mm, vias 0 -> 8
- net /R0: track 0.00 -> 51.7 mm
- net Net-(J1-~{RESET}): track 0.00 -> 40.0 mm
- net Net-(J1-SWDIO): track 0.00 -> 38.2 mm
- net GND: track 19.6 -> 46.6 mm, vias 10 -> 37
- net /R3: track 58.9 -> 85.7 mm
- net /R4: track 64.3 -> 90.3 mm
- net /R5: track 69.3 -> 94.9 mm
- net /R7: track 79.9 -> 104.9 mm
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- added copper zone on F.Cu, net GND
Other:
- outline, holes or cut-outs redrawn
- board text added: "Battery model: CR2032"
- board text added: "Electronic card 2025 V1.1 Art: Jordi Navarrete Electronics: Eric Navarrete"
- board text removed: "Battery model: CR2032 Insert with larger side up!"
- board text removed: "Electronic card 2024 V1 Art: Jordi Navarrete Electronics: Eric Navarrete"
