File: PCB/Chirstmas-Card.kicad_sch (KiCad schematic)
At the start: 100 parts, among them J1 Conn_ARM_SWD_TagConnect_TC203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, SW1 SW_SPST, SW2 SW_SPST, SW3 SW_SPST, U1 PAM8904EGPR, U2 STM32G030C6Tx, Y1 Crystal

Commit message: Added initial buzzer functionality
Parts:
- removed C1, C2: 10uF, Capacitor_SMD:C_0603_1608Metric, symbol Device:C_Small
- removed C3, C4: 1uF, Capacitor_SMD:C_0603_1608Metric, symbol Device:C_Small
- removed R1, R2, R3, R4, R5, R6, R7, R8: 0, Resistor_SMD:R_0402_1005Metric, symbol Device:R
- removed R10, R11, R15, R16: 0r, Resistor_SMD:R_0402_1005Metric, symbol Device:R
- removed R14: 100k, Resistor_SMD:R_0402_1005Metric, symbol Device:R
- removed U1: PAM8904EGPR, EN_Designs-Footprints:QFN50P300X300X100-13N, symbol EN_Designs-Symbols:PAM8904EGPR
- BT1: JLC (none) -> C70377; MPN (none) -> CR2032-BS-6-1
- C10, C7, C8, C9: JLC (none) -> C131394; MPN (none) -> CC0402KRX7R9BB104
- C11: JLC (none) -> C96446; MPN (none) -> CL10A106MA8NRNC
- C5, C6: JLC (none) -> C1548; MPN (none) -> 0402CG150J500NT
- D1, D10, D11, D12, D13, D14, D15, D16, D17, D18, D19, D2, D20, D21, D22, D23, D24, D25, D26, D27, D28, D29, D3, D30, D31, D32, D33, D34, D35, D36, D37, D38, D39, D4, D40, D41, D42, D43, D44, D45, D46, D47, D48, D49, D5, D50, D51, D52, D53, D54, D55, D56, D57, D58, D59, D6, D60, D61, D62, D63, D64, D7, D8, D9: footprint LED_SMD:LED_0805_2012Metric -> EN_Designs-Footprints:MHT151WDT; JLC (none) -> C401114; MPN (none) -> MHT151WDT
- J1: now not fitted
- LS1: JLC (none) -> C391037; MPN (none) -> FUET-1230
- R12, R13, R9: footprint Resistor_SMD:R_0402_1005Metric -> Resistor_SMD:R_0603_1608Metric; JLC (none) -> C25741; MPN (none) -> 0402WGF1003TCE
- SW1, SW2, SW3: JLC (none) -> C2837531; MPN (none) -> KH-6X6X5H-STM
- U2: JLC (none) -> C529328; MPN (none) -> STM32G030C6T6
- Y1: JLC (none) -> C32346; MPN (none) -> Q13FC1350000400
Connections:
- net BTN1: now also U2.39 (PD1); no longer U2.37 (PA15)
- net BTN3: now also U2.37 (PA15); no longer U2.39 (PD1)
- net C1: now also D14.2 (A), D22.2 (A), D30.2 (A), D38.2 (A), D46.2 (A), D54.2 (A), D6.2 (A), D62.2 (A), U2.24 (PB12); no longer U2.17 (PA6)
- net C2: now also D13.2 (A), D21.2 (A), D29.2 (A), D37.2 (A), D45.2 (A), D5.2 (A), D53.2 (A), D61.2 (A), U2.23 (PB11); no longer U2.18 (PA7)
- net C3: now also D12.2 (A), D20.2 (A), D28.2 (A), D36.2 (A), D4.2 (A), D44.2 (A), D52.2 (A), D60.2 (A), U2.22 (PB10); no longer U2.19 (PB0)
- net C4: now also D11.2 (A), D19.2 (A), D27.2 (A), D3.2 (A), D35.2 (A), D43.2 (A), D51.2 (A), D59.2 (A), U2.21 (PB2); no longer U2.20 (PB1)
- net C5: now also D10.2 (A), D18.2 (A), D2.2 (A), D26.2 (A), D34.2 (A), D42.2 (A), D50.2 (A), D58.2 (A), U2.20 (PB1); no longer U2.21 (PB2)
- net C6: now also D1.2 (A), D17.2 (A), D25.2 (A), D33.2 (A), D41.2 (A), D49.2 (A), D57.2 (A), D9.2 (A), U2.19 (PB0); no longer U2.22 (PB10)
- net C7: now also D16.2 (A), D24.2 (A), D32.2 (A), D40.2 (A), D48.2 (A), D56.2 (A), D64.2 (A), D8.2 (A), U2.18 (PA7); no longer U2.23 (PB11)
- net C8: now also D15.2 (A), D23.2 (A), D31.2 (A), D39.2 (A), D47.2 (A), D55.2 (A), D63.2 (A), D7.2 (A), U2.17 (PA6); no longer U2.24 (PB12)
- net at U2.42 (PB3): now also LS1.1
- net at U2.45 (PB6): now also LS1.2
- net BUZZER: no longer names the net of U2.15 (PA4)
Other:
- note added: "4u / (1 / 8M) = 32"
- moved on the sheet: BT1, LS1

Commit message: -migration to new cube mx version and cmake toolchain
Parts:
- removed R13, R9: 100k, Resistor_SMD:R_0603_1608Metric, symbol Device:R
- added R4, R5: 0, Resistor_SMD:R_0603_1608Metric, symbol Device:R
- renumbered C9 to C1, C10 to C2, C11 to C3, C8 to C4, C7 to C5, C5 to C7, D7 to D1, D16 to D10, D9 to D11, D10 to D12, D11 to D13, D12 to D14, D13 to D15, D14 to D16, D23 to D17, D24 to D18, D17 to D19, D8 to D2, D18 to D20, D19 to D21, D20 to D22, D21 to D23, D22 to D24, D31 to D25, D32 to D26, D25 to D27, D26 to D28, D27 to D29, D1 to D3, D28 to D30, D29 to D31, D30 to D32, D39 to D33, D40 to D34, D33 to D35, D34 to D36, D35 to D37, D36 to D38, D37 to D39, D2 to D4, D38 to D40, D47 to D41, D48 to D42, D41 to D43, D42 to D44, D43 to D45, D44 to D46, D45 to D47, D46 to D48, D55 to D49, D3 to D5, D56 to D50, D49 to D51, D50 to D52, D51 to D53, D52 to D54, D53 to D55, D54 to D56, D63 to D57, D64 to D58, D57 to D59, D4 to D6, D58 to D60, D59 to D61, D60 to D62, D61 to D63, D62 to D64, D5 to D7, D6 to D8, D15 to D9, R12 to R2, U2 to U1
Connections:
- net BTN2: now also U1.1 (PC13); no longer U1.44 (PB5)
- net C1: now also D10.2 (A), D18.2 (A), D2.2 (A), D26.2 (A), D34.2 (A), D42.2 (A), D50.2 (A), D58.2 (A), U1.12 (PA1); no longer D16.2 (A), D24.2 (A), D32.2 (A), D40.2 (A), D48.2 (A), D56.2 (A), D64.2 (A), D8.2 (A), U1.24 (PB12)
- net C2: now also D11.2 (A), D19.2 (A), D27.2 (A), D3.2 (A), D35.2 (A), D43.2 (A), D51.2 (A), D59.2 (A), U1.13 (PA2); no longer D15.2 (A), D23.2 (A), D31.2 (A), D39.2 (A), D47.2 (A), D55.2 (A), D63.2 (A), D7.2 (A), U1.23 (PB11)
- net C3: now also D12.2 (A), D20.2 (A), D28.2 (A), D36.2 (A), D4.2 (A), D44.2 (A), D52.2 (A), D60.2 (A), U1.14 (PA3); no longer D14.2 (A), D22.2 (A), D30.2 (A), D38.2 (A), D46.2 (A), D54.2 (A), D6.2 (A), D62.2 (A), U1.22 (PB10)
- net C4: now also U1.15 (PA4); no longer U1.21 (PB2)
- net C5: now also D14.2 (A), D22.2 (A), D30.2 (A), D38.2 (A), D46.2 (A), D54.2 (A), D6.2 (A), D62.2 (A), U1.16 (PA5); no longer D12.2 (A), D20.2 (A), D28.2 (A), D36.2 (A), D4.2 (A), D44.2 (A), D52.2 (A), D60.2 (A), U1.20 (PB1)
- net C6: now also D15.2 (A), D23.2 (A), D31.2 (A), D39.2 (A), D47.2 (A), D55.2 (A), D63.2 (A), D7.2 (A), U1.17 (PA6); no longer D11.2 (A), D19.2 (A), D27.2 (A), D3.2 (A), D35.2 (A), D43.2 (A), D51.2 (A), D59.2 (A), U1.19 (PB0)
- net C7: now also D16.2 (A), D24.2 (A), D32.2 (A), D40.2 (A), D48.2 (A), D56.2 (A), D64.2 (A), D8.2 (A); no longer D10.2 (A), D18.2 (A), D2.2 (A), D26.2 (A), D34.2 (A), D42.2 (A), D50.2 (A), D58.2 (A)
- net R1: now also D10.1 (K), D11.1 (K), D12.1 (K), D13.1 (K), D14.1 (K), D15.1 (K), D16.1 (K), D9.1 (K), U1.20 (PB1); no longer D1.1 (K), D2.1 (K), D3.1 (K), D4.1 (K), D5.1 (K), D6.1 (K), D7.1 (K), D8.1 (K), U1.25 (PB13)
- net R2: now also D17.1 (K), D18.1 (K), D19.1 (K), D20.1 (K), D21.1 (K), D22.1 (K), D23.1 (K), D24.1 (K), U1.21 (PB2); no longer D10.1 (K), D11.1 (K), D12.1 (K), D13.1 (K), D14.1 (K), D15.1 (K), D16.1 (K), D9.1 (K), U1.26 (PB14)
- net R3: now also D25.1 (K), D26.1 (K), D27.1 (K), D28.1 (K), D29.1 (K), D30.1 (K), D31.1 (K), D32.1 (K), U1.42 (PB3); no longer D17.1 (K), D18.1 (K), D19.1 (K), D20.1 (K), D21.1 (K), D22.1 (K), D23.1 (K), D24.1 (K), U1.27 (PB15)
- net R4: now also D33.1 (K), D34.1 (K), D35.1 (K), D36.1 (K), D37.1 (K), D38.1 (K), D39.1 (K), D40.1 (K), U1.43 (PB4); no longer D25.1 (K), D26.1 (K), D27.1 (K), D28.1 (K), D29.1 (K), D30.1 (K), D31.1 (K), D32.1 (K), U1.28 (PA8)
- net R5: now also D41.1 (K), D42.1 (K), D43.1 (K), D44.1 (K), D45.1 (K), D46.1 (K), D47.1 (K), D48.1 (K), U1.44 (PB5); no longer D33.1 (K), D34.1 (K), D35.1 (K), D36.1 (K), D37.1 (K), D38.1 (K), D39.1 (K), D40.1 (K), U1.29 (PA9/NC)
- net R6: now also D49.1 (K), D50.1 (K), D51.1 (K), D52.1 (K), D53.1 (K), D54.1 (K), D55.1 (K), D56.1 (K), U1.45 (PB6); no longer D41.1 (K), D42.1 (K), D43.1 (K), D44.1 (K), D45.1 (K), D46.1 (K), D47.1 (K), D48.1 (K), U1.30 (PC6)
- net R7: now also D57.1 (K), D58.1 (K), D59.1 (K), D60.1 (K), D61.1 (K), D62.1 (K), D63.1 (K), D64.1 (K), U1.46 (PB7); no longer D49.1 (K), D50.1 (K), D51.1 (K), D52.1 (K), D53.1 (K), D54.1 (K), D55.1 (K), D56.1 (K), U1.31 (PC7)
- net RESET: now also R5.2; no longer J1.3 (~{RESET})
- net SWDIO: now also R4.2; no longer J1.2 (SWDIO)
- net C0: now reaches U1.11 (PA0)
- net C0: now also D1.2 (A), D17.2 (A), D25.2 (A), D33.2 (A), D41.2 (A), D49.2 (A), D57.2 (A), D9.2 (A)
- net at LS1.1: now also U1.28 (PA8); no longer U1.42 (PB3)
- net at LS1.2: now also U1.29 (PA9/NC); no longer U1.45 (PB6)
- removed net C8: D1.2 (A), D17.2 (A), D25.2 (A), D33.2 (A), D41.2 (A), D49.2 (A), D57.2 (A), D9.2 (A), U1.17 (PA6)
- removed net R8: D57.1 (K), D58.1 (K), D59.1 (K), D60.1 (K), D61.1 (K), D62.1 (K), D63.1 (K), D64.1 (K), U1.32 (PA10/NC)
- new net: J1.2 (SWDIO), R4.1
- new net: J1.3 (~{RESET}), R5.1
- new net R0: D1.1 (K), D2.1 (K), D3.1 (K), D4.1 (K), D5.1 (K), D6.1 (K), D7.1 (K), D8.1 (K), U1.19 (PB0)
Other:
- moved on the sheet: C6, C7, LS1, R2, SW1, SW2, SW3, Y1
